File: working/spectrogram-left/spectrogram-left.kicad_pcb (KiCad board)
At the start: 2 copper layers, 135.7 x 99.4 mm, 107 parts, among them U2 ProMicro

Commit message: Upodated stuff, finalish version for left
Parts:
- removed the REF** at (56.9, 69.3)
- removed the REF** at (112.9, 37.3)
- removed the REF** at (96.1, 28.3)
- removed the REF** at (82.6, 31.5)
- removed the REF** at (93.7, 37.3)
- removed the REF** at (66.3, 41.8)
- removed the REF** at (79.2, 41.0)
- removed the REF** at (47.9, 48.7)
- removed the REF** at (40.2, 40.3)
- removed the REF** at (147.7, 75.6)
- removed the REF** at (64.3, 37.4)
- removed the REF** at (63.4, 31.5)
- removed the REF** at (44.8, 30.6)
- removed the REF** at (65.1, 51.2)
- removed the REF** at (62.0, 48.6)
- removed the REF** at (104.0, 111.0)
- removed the REF** at (107.0, 105.8)
- removed the REF** at (126.0, 38.7)
- removed the REF** at (124.1, 36.8)
- removed the REF** at (147.8, 67.9)
- removed the REF** at (133.8, 37.3)
- removed the REF** at (67.3, 47.0)
- removed the REF** at (72.7, 45.0)
- removed the REF** at (69.6, 45.6)
- removed the REF** at (82.0, 37.0)
- removed the REF** at (96.9, 109.6)
- removed the REF** at (57.7, 41.4)
- removed the REF** at (139.2, 61.9)
- removed the REF** at (142.8, 55.2)
- removed the REF** at (143.5, 49.8)
- removed the REF** at (110.8, 45.1)
- removed the REF** at (148.0, 38.0)
- removed TP2: C6, Keebio-Parts:SinglePad
- SW_D1: footprint jakestuff:ChocMX_sameside_flippedpads_2.25U_flippedstab -> jakestuff:ChocMX_2.25U_reversedstab
- U2: footprint Keebio-Parts:ArduinoProMicro -> Keebio-Parts:ArduinoProMicro-ZigZag
- moved REF** 15.9 mm to (128.0, 49.5)
- moved REF** 10.6 mm to (99.0, 47.5)
- moved D_B4 9.37 mm to (108.8, 61.8)
- moved D_B5 9.36 mm to (127.4, 61.8)
- moved D_B6 9.36 mm to (129.8, 61.8)
- moved D_B3 9.12 mm to (89.0, 61.5)
- moved D_B2 9.12 mm to (70.0, 61.5)
- moved D_B1 9.11 mm to (72.5, 61.5)
- moved U2 1.57 mm to (39.0, 50.8)
- moved D_E2 0.27 mm to (71.5, 109.7)
Routing:
- net Col7: track 0.00 -> 217.0 mm, vias 0 -> 11
- net Col5: track 0.00 -> 192.7 mm, vias 0 -> 13
- net Col6: track 0.00 -> 160.0 mm, vias 0 -> 9
- net RowE: track 0.00 -> 151.7 mm, vias 0 -> 5
- net RowD: track 0.00 -> 129.6 mm, vias 0 -> 6
- net Col4: track 0.00 -> 127.4 mm, vias 0 -> 8
- net Col3: track 0.00 -> 126.4 mm, vias 0 -> 9
- net Col1: track 0.00 -> 121.1 mm, vias 0 -> 13
- net RowC: track 0.00 -> 110.0 mm, vias 0 -> 7
- net Col2: track 0.00 -> 102.5 mm, vias 0 -> 8
- net RowA: track 0.00 -> 100.5 mm, vias 0 -> 6
- net RowB: track 0.00 -> 96.0 mm, vias 0 -> 5
- net Net-(D_E7-A): track 0.00 -> 55.8 mm, vias 0 -> 5
- net Net-(D_A7-A): track 0.00 -> 52.1 mm, vias 0 -> 3
- net Net-(D_E5-A): track 0.00 -> 47.9 mm, vias 0 -> 5
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Other:
- board size 135.7 x 99.4 mm -> 135.7 x 91.1 mm
