File: working/spectrogram-left/spectrogram-left.kicad_pcb (KiCad board)
At the start: 2 copper layers, 135.7 x 91.1 mm, 74 parts, among them U2 ProMicro

Commit message: Pushed updtes
Parts:
- added ?: , , F.Cu at (28.0, 40.5)
- added ?: , , F.Cu at (54.0, 99.0)
- added ?: , , F.Cu at (128.0, 52.0)
- added ?: , , F.Cu at (41.0, 55.0)
- added ?: , , F.Cu at (39.0, 61.5)
- added ?: , , F.Cu at (51.0, 100.0)
- SW_EB7: footprint jakestuff:ChocMX_flippedpads_2.25U_reversedstab -> jakestuff:ChocMX_flippedpads_2.25U
- moved REF** 10.5 mm to (89.5, 52.0)
- moved REF** 2.44 mm to (87.5, 57.0)
- moved D_A2 2.36 mm to (56.0, 44.1), turned to 90 degrees
- moved D_E7 1.25 mm to (130.0, 109.2)
- moved D_E5 1.00 mm to (127.5, 109.2)
- moved D_D3 0.50 mm to (85.0, 90.0)
- turned SW_EB7 to 180 degrees
Routing:
- net Col7: track 217.0 -> 196.4 mm, vias 11 -> 8
- net GND: track 0.00 -> 12.3 mm
- net (no net): track 0.00 -> 7.33 mm
- net Net-(D_E7-A): track 55.8 -> 50.3 mm
- net Net-(D_A2-A): track 20.0 -> 15.4 mm
- net Net-(D_E5-A): track 47.9 -> 46.9 mm
- net RowD: track 129.6 -> 130.5 mm
- net RowA: track 100.5 -> 101.3 mm
- net RowE: track 151.7 -> 151.0 mm
- net Net-(D_B1-A): track 34.6 -> 35.1 mm
- net Net-(D_D3-A): track 16.7 -> 16.2 mm
