File: working/spectrogram-left/spectrogram-left.kicad_sch (KiCad schematic)
At the start: 70 parts, among them U2 ProMicro

Commit message: swapped left side footprints, still have to route
Parts:
- SW_E5: footprint jakestuff:ChocMX_flippedpads_2.25U -> jakestuff:ChocMX_flippedpads_2.25U_reversedstab
- SW_EB5: footprint jakestuff:ChocMX -> jakestuff:ChocMX_flippedpads
Changed lines of the file:
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@@
 			)
 		)
-		(property "Footprint" "jakestuff:ChocMX_flippedpads_2.25U"
+		(property "Footprint" "jakestuff:ChocMX_flippedpads_2.25U_reversedstab"
 			(at 165.1 96.52 0)
 			(effects
@@
 			)
 		)
-		(property "Footprint" "jakestuff:ChocMX"
+		(property "Footprint" "jakestuff:ChocMX_flippedpads"
 			(at 165.1 104.14 0)
 			(effects

Commit message: Upodated stuff, finalish version for left
Parts:
- SW_D1: footprint jakestuff:ChocMX_sameside_flippedpads_2.25U_flippedstab -> jakestuff:ChocMX_2.25U_reversedstab
- U2: footprint Keebio-Parts:ArduinoProMicro -> Keebio-Parts:ArduinoProMicro-ZigZag
Changed lines of the file:
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@@
 			)
 		)
-		(property "Footprint" "Keebio-Parts:ArduinoProMicro"
+		(property "Footprint" "Keebio-Parts:ArduinoProMicro-ZigZag"
 			(at 80.01 107.95 90)
 			(effects
@@
 			)
 		)
-		(property "Footprint" "jakestuff:ChocMX_sameside_flippedpads_2.25U_flippedstab"
+		(property "Footprint" "jakestuff:ChocMX_2.25U_reversedstab"
 			(at 104.14 78.74 0)
 			(effects
