File: working/spectrogram-left/spectrogram-left.kicad_sch (KiCad schematic)
At the start: 70 parts, among them U2 ProMicro

Commit message: Pushed updtes
Parts:
- SW_EB7: footprint jakestuff:ChocMX_flippedpads_2.25U_reversedstab -> jakestuff:ChocMX_flippedpads_2.25U
Changed lines of the file:
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@@
 			)
 		)
-		(property "Footprint" "jakestuff:ChocMX_flippedpads_2.25U_reversedstab"
+		(property "Footprint" "jakestuff:ChocMX_flippedpads_2.25U"
 			(at 195.58 104.14 0)
 			(effects
