File: working/spectrogram-left/spectrogram-left-bottom.kicad_pcb (KiCad board)
At the start: 2 copper layers, 146.1 x 111.2 mm, 9 parts, among them U3 HOLE

Commit message: Pushed updtes
Parts:
- removed G***: LOGO, Keebio-Art:Keebio-TwoTone
- removed U3: HOLE, Keebio-Parts:SolidCopper
Other:
- net class Default removed
- net class Power Tracks removed
- board text added: "~"
- board text added: "、"
- board text added: "ノ"
- board text added: "／l （ﾟ ｡ ７ l ~ヽ じしf_,)"
- board text added: "／l （ﾟ､ ｡ ７ l ~ヽ じしf_,)"
