File: working/spectrogram-left/spectrogram-left-top.kicad_pcb (KiCad board)
At the start: 2 copper layers, 146.1 x 111.2 mm, 7 parts

Commit message: Pushed updtes
Other:
- outline, holes or cut-outs redrawn
- net class Default removed
- net class Power Tracks removed
